File: PCB/_autosave-PCB.kicad_pcb (KiCad board)
At the start: 2 copper layers, 8 parts, among them J1 Barrel_Jack_MountingPin, M1 Motor_Servo, M2 Motor_Servo, M3 Motor_Servo, M4 Motor_Servo, M5 Motor_Servo, M6 Motor_Servo, U1 ESP32-Devkit-V1

Commit message: PCB
Parts:
- J1: footprint Connector_BarrelJack:BarrelJack_CUI_PJ-063AH_Horizontal_CircularHoles -> Connector_BarrelJack:BarrelJack_CUI_PJ-102AH_Horizontal
- moved M4 47.9 mm to (126.9, 115.7), turned to 90 degrees
- moved M1 43.8 mm to (93.0, 120.8), turned to -90 degrees
- moved M2 41.8 mm to (92.9, 124.8), turned to -90 degrees
- moved M3 39.4 mm to (92.7, 129.4), turned to -90 degrees
- moved J1 24.5 mm to (154.3, 101.7), turned to 90 degrees
- moved M6 15.9 mm to (92.6, 112.1), turned to -90 degrees
- moved M5 13.2 mm to (92.7, 116.6), turned to -90 degrees
Routing:
- net PWM6: track 88.4 -> 4.68 mm
- net PWM5: track 23.3 -> 5.82 mm
- net PWM4: track 18.9 -> 6.05 mm
- net PWM2: track 0.00 -> 6.10 mm
- net PWM1: track 0.00 -> 4.45 mm
- net PWM3: track 0.00 -> 3.82 mm
